File: Hardware/SparkFun_Pulse_Oximeter_Heart-Rate_Sensor.sch (EAGLE design)
At the start: 34 parts, among them U1 MAX30101EFD, U2 MAX32664GWEA, U3 1.8V/100mA, Y1 32.768kHz

Commit message: Clarifies "Address" text underneath MAX32664 symbol in schematic by adding "I2C"
Other:
- note added: "I2C Address: 0x55"
- note removed: "Address: 0x55"
Changed lines of the file:
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@@
 <text x="238.76" y="7.62" size="2.54" layer="94" font="vector">v01</text>
 <text x="139.7" y="167.64" size="1.27" layer="97" font="vector">VCC Range: 1.71 - 3.63V</text>
-<text x="142.24" y="116.84" size="1.27" layer="97" font="vector">Address: 0x55</text>
+<text x="139.7" y="116.84" size="1.27" layer="97" font="vector">I2C Address: 0x55</text>
 <wire x1="0" y1="111.76" x2="104.14" y2="111.76" width="0.2032" layer="97" style="shortdash"/>
 <wire x1="104.14" y1="111.76" x2="193.04" y2="111.76" width="0.2032" layer="97" style="shortdash"/>
