File: Hardware/SparkFun_Pulse_Oximeter_Heart-Rate_Sensor.sch (EAGLE design)
At the start: 34 parts, among them U1 MAX30101EFD, U2 MAX32664GWEA, U3 1.8V/100mA, Y1 32.768kHz

Commit message: Updates silk, updates bio sensor hub to slightly improved package, rolls version to v11
* Updates schematic to include part numbers on all parts
* Updates notes on parts
* Updates package size on 0402 components to 0402-tight
* Adds more vias
* Adds more measures
Parts:
- removed JP1: JUMPER-SMT_3_2-NC_TRACE_SILK, SparkFun-Jumpers:JUMPER-SMT_3_2-NC_TRACE_SILK
- added I2C: JUMPER-SMT_3_2-NC_TRACE_SILK, SparkFun-Jumpers:JUMPER-SMT_3_2-NC_TRACE_SILK
- added LOGO5: QWIIC_LOGO_4MM, SparkFun-Aesthetics:QWIIC_LOGO_4MM
- C2: device SparkFun-Capacitors:0.1UF-0402-16V-10% -> SparkFun-Capacitors:0.1UF-0402T-16V-10%
- C6, C7: device SparkFun-Capacitors:1.0UF-0402-16V-10% -> SparkFun-Capacitors:1.0UF-0402T-16V-10%
- J1, J2: value (none) -> QWIIC_RIGHT_ANGLE
- R4: value 100K -> 100k; device SparkFun-Resistors:100KOHM-0402-1/16W-1% -> SparkFun-Resistors:100KOHM-0402T-1/16W-1%
Connections:
- net 3.3V: now also I2C.2; no longer JP1.2
- net N$4: now also I2C.3; no longer JP1.3
- net N$5: now also I2C.1; no longer JP1.1
Other:
- note added: "1.8V VREG - SP6214"
- note added: "Cut jumpers to remove I2C Pullups."
- note added: "DC-DC Converter - PAM2401"
- note added: "Unshifted 7-bit Address: 0x55"
- note added: "Unshifted 7-bit Address: 0x57"
- note added: "VCC Range: 1-4.75V"
- note added: "VCC Range: 2.5 - 7V IOUT MAX: 100mA"
- note added: "v11"
- note removed: "1.8V VREG"
- note removed: "DC-DC Converter"
- note removed: "I2C Address: 0x55"
- note removed: "I2C Read Address: 0xAA I2C Write Address: 0xAB"
- note removed: "v01"
- moved on the sheet: C2, C6, C7, J4, R2, R5, R6, R7, Y1
